File: filter.kicad_sch (KiCad schematic)
At the start: 91 parts, among them U1 ${SIM.PARAMS}

Commit message: Upgrade
Parts:
- removed C10, C11, C19, C20: C,IEC, symbol PCM_Generic-50:C,IEC
- removed C14, C15, C18, C9: C,IEC, symbol PCM_Generic:C,IEC
- removed R11, R12, R13, R17, R18, R22, R24, R25, R26, R30, R31, R33, R5: R,IEC, symbol PCM_Generic:R,IEC
- added C27, C28: C,IEC, symbol PCM_Generic:C,IEC
- added R4: R HF, symbol PCM_Generic:R,IEC
- R19: value R HF ,IEC -> R HF
Connections:
- net at C23.2 (-), C24.1 (+): now also C16.2 (-), C17.2 (-), R20.1 (+), R21.1 (+)
- net at C4.2 (-), C5.1 (+): now also C1.2 (-), C6.2 (-), R10.1 (+), R3.1 (+)
- net at C25.2 (-), C26.1 (+): now also R19.1 (+)
- new net: C27.2 (-), C28.1 (+), R4.1 (+)
Other:
- note added: "04.09.2023"
- note added: "6 cm"
- note added: "OSH License"
- note removed: "Must be OSHW"
- moved on the sheet: R19

Commit message: Upgrade
Parts:
- added C10, C9: C,IEC, symbol PCM_Generic:C,IEC
- added L1: L 1,ferrite-bead,IEC, symbol PCM_Generic:L,ferrite-bead,IEC
- added L2, L3, L4: L 1, ferrite-bead,IEC, symbol PCM_Generic:L,ferrite-bead,IEC
- added R11, R12, R13, R18, R22, R7: 8 Om, symbol PCM_Generic:R,IEC
- added R15, R17, R5, R6: 10 Om, symbol PCM_Generic:R,IEC
Connections:
- net at C16.2 (-), C17.2 (-), R20.1 (+)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: now also R5.1 (+), R6.1 (+); no longer C23.2 (-), C24.1 (+)
- net at C1.2 (-), C6.2 (-), R10.1 (+)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: now also R15.1 (+), R17.1 (+); no longer C4.2 (-), C5.1 (+)
- net at C21.1 (+), R27.1 (+): now also L1.1 (+)
- net at C3.1 (+), R2.1 (+): now also L3.1 (+)
- net at C22.1 (+), R29.1 (+): now also L2.1 (+)
- net at C8.1 (+), R9.1 (+): now also L4.1 (+)
- new net: C23.2 (-), C24.1 (+), R11.1 (+), R7.1 (+)
- new net: C4.2 (-), C5.1 (+), R12.1 (+), R13.1 (+)
- new net: R12.2 (-), R13.2 (-), R15.2 (-), R17.2 (-)
- new net: C10.1 (+), C9.2 (-), R18.1 (+), R22.1 (+)
- new net: R18.2 (-), R22.2 (-)
- new net: R11.2 (-), R5.2 (-), R6.2 (-), R7.2 (-)
Other:
- note added: "Updated on 10/10/2023"
- note removed: "6 cm"

Commit message: Upgrade
Parts:
- L3, L4: value L 1, ferrite-bead,IEC -> L 2, ferrite-bead,IEC
Changed lines of the file:
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@@
       (effects (font (size 2.54 2.54)) (justify left))
     )
-    (property "Value" "L 1, ferrite-bead,IEC" (at 134.62 81.2799 0)
+    (property "Value" "L 2, ferrite-bead,IEC" (at 134.62 81.2799 0)
       (effects (font (size 2.54 2.54)) (justify left))
     )
@@
       (effects (font (size 2.54 2.54)) (justify left))
     )
-    (property "Value" "L 1, ferrite-bead,IEC" (at 200.66 68.5799 0)
-      (effects (font (size 2.54 2.54)) (justify left))
-    )
+    (property "Value" "L 2, ferrite-bead,IEC" (at 200.66 68.5799 0)
+      (effects (font (size 2.54 2.54)) (justify left))
+    )

Commit message: Upgrade
Parts:
- added R23, R24: 8 Om, symbol PCM_Generic:R,IEC
Connections:
- new net: R23.1 (+), R24.1 (+)
- new net: R23.2 (-), R24.2 (-)
Other:
- note added: "13"
- note added: "Updated 2023.10.23"
- note removed: "12"
Changed lines of the file:
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@@
   (junction (at 398.78 31.75) (diameter 0) (color 0 0 0 0)
   )
+  (junction (at 132.08 116.84) (diameter 0) (color 0 0 0 0)
+  )
   (junction (at 72.39 60.96) (diameter 0) (color 0 0 0 0)
   )
@@
   (junction (at 196.85 125.73) (diameter 0) (color 0 0 0 0)
   )
+  (junction (at 132.08 127) (diameter 0) (color 0 0 0 0)
+  )
   (junction (at 410.21 31.75) (diameter 0) (color 0 0 0 0)
   )
@@
   (junction (at 457.2 31.75) (diameter 0) (color 0 0 0 0)
   )
+  (wire (pts (xy 132.08 127) (xy 143.51 127))
+    (stroke (width 0) (type default))
+  )
   (wire (pts (xy 132.08 33.02) (xy 132.08 39.37))
     (stroke (width 0) (type default))
@@
     (stroke (width 0) (type default))
   )
+  (wire (pts (xy 132.08 116.84) (xy 143.51 116.84))
+    (stroke (width 0) (type default))
+  )
   (wire (pts (xy 146.05 19.05) (xy 146.05 39.37))
     (stroke (width 0) (type default))
@@
     (stroke (width 0) (type default))
   )
+  (wire (pts (xy 128.27 127) (xy 132.08 127))
+    (stroke (width 0) (type default))
+  )
   (wire (pts (xy 58.42 60.96) (xy 58.42 22.86))
     (stroke (width 0) (type default))
@@
     (stroke (width 0) (type default))
   )
+  (wire (pts (xy 128.27 116.84) (xy 132.08 116.84))
+    (stroke (width 0) (type default))
+  )
   (wire (pts (xy 438.15 69.85) (xy 438.15 63.5))
     (stroke (width 0) (type default))
@@
     (stroke (width 0) (type default))
   )
-  (wire (pts (xy 132.08 97.79) (xy 132.08 129.54))
+  (wire (pts (xy 412.75 106.68) (xy 415.29 106.68))
     (stroke (width 0) (type default))
   )
-  (wire (pts (xy 412.75 106.68) (xy 415.29 106.68))
+  (wire (pts (xy 132.08 127) (xy 132.08 129.54))
     (stroke (width 0) (type default))
   )
@@
     (stroke (width 0) (type default))
   )
+  (wire (pts (xy 132.08 97.79) (xy 132.08 116.84))
+    (stroke (width 0) (type default))
+  )
   (wire (pts (xy 459.74 95.25) (xy 459.74 106.68))
     (stroke (width 0) (type default))
@@
     (effects (font (face "KiCad Font") (size 1.9 1.9)) (justify left))
   )
+  (text "Updated 2023.10.23\n" (at 242.57 170.18 0)
+    (effects (font (size 1.27 1.27)) (justify left bottom))
+  )
   (text "Filter" (at 186.69 190.5 0)
     (effects (font (size 1.27 1.27)) (justify left bottom))
@@
     (effects (font (size 1.27 1.27)) (justify left bottom))
   )
-  (text "12" (at 270.51 194.31 0)
+  (text "13" (at 270.51 194.31 0)
     (effects (font (size 1.27 1.27)) (justify left bottom))
   )
@@
     )
   )
+  (symbol (lib_id "PCM_Generic:R,IEC") (at 128.27 121.92 0) (unit 1)
+    (in_bom yes) (on_board yes) (dnp no) (fields_autoplaced)
+    (property "Reference" "R23" (at 130.81 119.3799 0)
+      (effects (font (size 2.54 2.54)) (justify left))
+    )
+    (property "Value" "8 Om" (at 130.81 124.4599 0)
+      (effects (font (size 2.54 2.54)) (justify left))
+    )
+    (property "Footprint" "" (at 128.27 121.92 0)
+      (effects (font (size 2.54 2.54)) hide)
+    )
+    (property "Datasheet" "" (at 128.27 121.92 0)
+      (effects (font (size 2.54 2.54)) hide)
+    )
+    (property "Indicator" "" (at 125.73 119.38 0)
+      (effects (font (size 1.27 1.27)) hide)
+    )
+    (pin "1")
+    (pin "2")
+    (instances
+      (project "filter"
+        (path "/69b3d959-9103-4d24-8a1d-6bf78309c8d1"
+          (reference "R23") (unit 1)
+        )
+      )
+    )
+  )
   (symbol (lib_id "PCM_Generic:R,IEC") (at 132.08 52.07 0) (mirror x) (unit 1)
     (in_bom yes) (on_board yes) (dnp no) (fields_autoplaced)
@@
         )
       )
+    )
+  )
+  (symbol (lib_id "PCM_Generic:R,IEC") (at 143.51 121.92 0) (unit 1)
+    (in_bom yes) (on_board yes) (dnp no) (fields_autoplaced)
+    (property "Reference" "R24" (at 146.05 119.3799 0)
+      (effects (font (size 2.54 2.54)) (justify left))
+    )
+    (property "Value" "8 Om" (at 146.05 124.4599 0)
+      (effects (font (size 2.54 2.54)) (justify left))
+    )
+    (property "Footprint" "" (at 143.51 121.92 0)
+      (effects (font (size 2.54 2.54)) hide)
+    )
+    (property "Datasheet" "" (at 143.51 121.92 0)
+      (effects (font (size 2.54 2.54)) hide)
+    )
+    (property "Indicator" "" (at 140.97 119.38 0)
+      (effects (font (size 1.27 1.27)) hide)
+    )
+    (pin "1")
+    (pin "2")
+    (instances
+      (project "filter"
+        (path "/69b3d959-9103-4d24-8a1d-6bf78309c8d1"
+          (reference "R24") (unit 1)
+        )
+      )

Commit message: Upgrade
Parts:
- removed R11, R13, R18, R24: 8 Om, symbol PCM_Generic:R,IEC
Other:
- note added: "29.02.2024"
- note added: "Same filters at 1.5-2 Km distance"
- moved on the sheet: R12, R22, R23, R7

Commit message: Upgrade
Parts:
- added C11, C14: C,22pF, symbol PCM_Generic:C,IEC
- added R11: 90 Om, symbol PCM_Generic:R,IEC
Connections:
- new net: C11.2 (-), C14.1 (+), R11.1 (+)
Changed lines of the file:
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@@
   (junction (at 198.12 39.37) (diameter 0) (color 0 0 0 0)
   )
+  (junction (at 205.74 144.78) (diameter 0) (color 0 0 0 0)
+  )
   (junction (at 90.17 22.86) (diameter 0) (color 0 0 0 0)
   )
@@
     (stroke (width 0) (type default))
   )
+  (wire (pts (xy 203.2 134.62) (xy 203.2 83.82))
+    (stroke (width 0) (type default))
+  )
   (wire (pts (xy 488.95 31.75) (xy 488.95 53.34))
     (stroke (width 0) (type default))
   )
+  (wire (pts (xy 222.25 156.21) (xy 222.25 113.03))
+    (stroke (width 0) (type default))
+  )
   (wire (pts (xy 182.88 97.79) (xy 165.1 97.79))
     (stroke (width 0) (type default))
@@
     (stroke (width 0) (type default))
   )
+  (wire (pts (xy 186.69 133.35) (xy 182.88 133.35))
+    (stroke (width 0) (type default))
+  )
+  (wire (pts (xy 205.74 156.21) (xy 222.25 156.21))
+    (stroke (width 0) (type default))
+  )
   (wire (pts (xy 515.62 54.61) (xy 509.27 54.61))
     (stroke (width 0) (type default))
@@
     (stroke (width 0) (type default))
   )
+  (wire (pts (xy 201.93 144.78) (xy 205.74 144.78))
+    (stroke (width 0) (type default))
+  )
   (wire (pts (xy 459.74 69.85) (xy 454.66 69.85))
     (stroke (width 0) (type default))
@@
     (stroke (width 0) (type default))
   )
+  (wire (pts (xy 205.74 134.62) (xy 203.2 134.62))
+    (stroke (width 0) (type default))
+  )
   (wire (pts (xy 163.83 30.48) (xy 171.45 30.48))
     (stroke (width 0) (type default))
@@
     (stroke (width 0) (type default))
   )
+  (wire (pts (xy 191.77 144.78) (xy 186.69 144.78))
+    (stroke (width 0) (type default))
+  )
   (wire (pts (xy 171.45 44.45) (xy 160.02 44.45))
     (stroke (width 0) (type default))
@@
     (stroke (width 0) (type default))
   )
+  (wire (pts (xy 205.74 144.78) (xy 205.74 146.05))
+    (stroke (width 0) (type default))
+  )
   (wire (pts (xy 132.08 39.37) (xy 132.08 46.99))
     (stroke (width 0) (type default))
@@
     (stroke (width 0) (type default))
   )
+  (wire (pts (xy 186.69 144.78) (xy 186.69 133.35))
+    (stroke (width 0) (type default))
+  )
   (wire (pts (xy 438.15 69.85) (xy 438.15 63.5))
     (stroke (width 0) (type default))
@@
     )
   )
+  (symbol (lib_id "PCM_Generic:R,IEC") (at 196.85 144.78 270) (unit 1)
+    (in_bom yes) (on_board yes) (dnp no) (fields_autoplaced)
+    (property "Reference" "R11" (at 196.85 134.62 90)
+      (effects (font (size 2.54 2.54)))
+    )
+    (property "Value" "90 Om" (at 196.85 139.7 90)
+      (effects (font (size 2.54 2.54)))
+    )
+    (property "Footprint" "" (at 196.85 144.78 0)
+      (effects (font (size 2.54 2.54)) hide)
+    )
+    (property "Datasheet" "" (at 196.85 144.78 0)
+      (effects (font (size 2.54 2.54)) hide)
+    )
+    (property "Indicator" "" (at 199.39 142.24 0)
+      (effects (font (size 1.27 1.27)) hide)
+    )
+    (pin "1")
+    (pin "2")
+    (instances
+      (project "filter"
+        (path "/69b3d959-9103-4d24-8a1d-6bf78309c8d1"
+          (reference "R11") (unit 1)
+        )
+      )
+    )
+  )
   (symbol (lib_id "PCM_Generic:R,IEC") (at 444.5 90.17 0) (mirror y) (unit 1)
     (in_bom yes) (on_board yes) (dnp no) (fields_autoplaced)
@@
     )
   )
+  (symbol (lib_id "PCM_Generic:C,IEC") (at 205.74 151.13 0) (mirror y) (unit 1)
+    (in_bom yes) (on_board yes) (dnp no)
+    (property "Reference" "C14" (at 209.55 148.59 0)
+      (effects (font (size 2.54 2.54)) (justify right))
+    )
+    (property "Value" "C,22pF" (at 209.55 152.4 0)
+      (effects (font (size 2.54 2.54)) (justify right))
+    )
+    (property "Footprint" "" (at 205.74 151.13 0)
+      (effects (font (size 2.54 2.54)) hide)
+    )
+    (property "Datasheet" "" (at 205.74 151.13 0)
+      (effects (font (size 2.54 2.54)) hide)
+    )
+    (property "Indicator" "" (at 209.55 155.575 0)
+      (effects (font (size 1.27 1.27)) (justify right))
+    )
+    (property "Field5" "" (at 205.74 151.13 0)
+      (effects (font (size 1.27 1.27)) hide)
+    )
+    (pin "1")
+    (pin "2")
+    (instances
+      (project "filter"
+        (path "/69b3d959-9103-4d24-8a1d-6bf78309c8d1"
+          (reference "C14") (unit 1)
+        )
+      )
+    )
+  )
   (symbol (lib_id "PCM_Generic:R,IEC") (at 67.31 39.37 0) (unit 1)
     (in_bom yes) (on_board yes) (dnp no) (fields_autoplaced)
@@
         )
       )
+    )
+  )
+  (symbol (lib_id "PCM_Generic:C,IEC") (at 205.74 139.7 0) (mirror y) (unit 1)
+    (in_bom yes) (on_board yes) (dnp no)
+    (property "Reference" "C11" (at 209.55 137.16 0)
+      (effects (font (size 2.54 2.54)) (justify right))
+    )
+    (property "Value" "C,22pF" (at 209.55 140.97 0)
+      (effects (font (size 2.54 2.54)) (justify right))
+    )
+    (property "Footprint" "" (at 205.74 139.7 0)
+      (effects (font (size 2.54 2.54)) hide)
+    )
+    (property "Datasheet" "" (at 205.74 139.7 0)
+      (effects (font (size 2.54 2.54)) hide)
+    )
+    (property "Indicator" "" (at 209.55 144.145 0)
+      (effects (font (size 1.27 1.27)) (justify right))
+    )
+    (property "Field5" "" (at 205.74 139.7 0)
+      (effects (font (size 1.27 1.27)) hide)
+    )
+    (pin "1")
+    (pin "2")
+    (instances
+      (project "filter"
+        (path "/69b3d959-9103-4d24-8a1d-6bf78309c8d1"
+          (reference "C11") (unit 1)
+        )
+      )

Commit message: Upgrade
Parts:
- added C15: 1uF, symbol PCM_Elektuur:C
- added R13: 8 Om, symbol PCM_Elektuur:R
Connections:
- net PE: now also C15.1 (+), R13.1 (+)
- new net: C15.2 (-), R13.2 (-)
Other:
- note added: "They say this is idea from life of Tupak -_^^_-"
Changed lines of the file:
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@@
   (junction (at 472.44 31.75) (diameter 0) (color 0 0 0 0)
   )
+  (junction (at 172.72 147.32) (diameter 0) (color 0 0 0 0)
+  )
   (junction (at 457.2 31.75) (diameter 0) (color 0 0 0 0)
   )
@@
     (stroke (width 0) (type default))
   )
+  (wire (pts (xy 165.1 185.42) (xy 165.1 186.69))
+    (stroke (width 0) (type default))
+  )
   (wire (pts (xy 210.82 39.37) (xy 210.82 19.05))
     (stroke (width 0) (type default))
@@
     (stroke (width 0) (type default))
   )
+  (wire (pts (xy 165.1 165.1) (xy 165.1 147.32))
+    (stroke (width 0) (type default))
+  )
   (wire (pts (xy 381 83.82) (xy 381 69.85))
     (stroke (width 0) (type default))
@@
     (stroke (width 0) (type default))
   )
+  (wire (pts (xy 172.72 147.32) (xy 172.72 153.67))
+    (stroke (width 0) (type default))
+  )
   (wire (pts (xy 417.83 53.34) (xy 415.29 53.34))
     (stroke (width 0) (type default))
@@
     (stroke (width 0) (type default))
   )
-  (wire (pts (xy 172.72 144.78) (xy 172.72 153.67))
+  (wire (pts (xy 172.72 144.78) (xy 172.72 147.32))
     (stroke (width 0) (type default))
   )
@@
     (stroke (width 0) (type default))
   )
+  (wire (pts (xy 165.1 147.32) (xy 172.72 147.32))
+    (stroke (width 0) (type default))
+  )
   (wire (pts (xy 462.28 31.75) (xy 462.28 43.18))
     (stroke (width 0) (type default))
@@
   )
   (text_box "R1,R2,R8,R9,R12,R11,R16,R14,R27,R29,R25,R24 = 33KOm\nR3,R10,R13,R26,R21,R20 = 15KOm\nR4,R7,R15,R23,R30,R31,R33,R34,R35,R36 = 2-10MOm all dumping resistors must have same nominal ( 10MOm as example ) and model !!!!!\nR5,R6,R18,R15,R17,R22,R28,R32 = 7-10Om   R4,R19 = 50Om 2GHz about 450 W\nC1,C6,C9,C17,C16,C18 = 220nF\nC2,C3,C7,C8,C11,C10,C12,C13,C20,C19,C21,C22 = 100nF\nC15,C14 = 10-100 nF - optional, I use MC1230 | C4,C5 = 100 nF   C23,C24 = 35 mkF\nC25,C26, C27,C28 = 22 pF C9, C10 = 10 nF\n\ntry to keep maximum possible distance between filters ~ 30cm\n\nMC 1230 optional"
-    (at 16.51 149.86 0) (size 143.51 43.18)
+    (at 13.97 152.4 0) (size 143.51 43.18)
     (stroke (width 0) (type default))
     (fill (type none))
@@
     (effects (font (size 1.27 1.27)) (justify left bottom))
   )
+  (text "They say this is idea from life of Tupak -_^^_-" (at 158.75 165.1 0)
+    (effects (font (size 1.27 1.27)) (justify left bottom))
+  )
   (text "OSH License" (at 269.24 177.8 0)
     (effects (font (size 1.27 1.27)) (justify left bottom))
@@
     )
   )
+  (symbol (lib_id "PCM_Generic:P,PE") (at 165.1 186.69 0) (unit 1)
+    (in_bom yes) (on_board yes) (dnp no) (fields_autoplaced)
+    (property "Reference" "#PWR04" (at 168.91 182.88 0)
+      (effects (font (size 2.54 2.54)) (justify left) hide)
+    )
+    (property "Value" "P,PE" (at 168.91 186.69 0)
+      (effects (font (size 0 0)) (justify left) hide)
+    )
+    (property "Footprint" "" (at 165.1 186.69 0)
+      (effects (font (size 2.54 2.54)) hide)
+    )
+    (property "Datasheet" "" (at 165.1 186.69 0)
+      (effects (font (size 2.54 2.54)) hide)
+    )
+    (pin "0")
+    (instances
+      (project "filter"
+        (path "/69b3d959-9103-4d24-8a1d-6bf78309c8d1"
+          (reference "#PWR04") (unit 1)
+        )
+      )
+    )
+  )
   (symbol (lib_id "PCM_Generic:R,IEC") (at 125.73 105.41 0) (unit 1)
     (in_bom yes) (on_board yes) (dnp no) (fields_autoplaced)
@@
     )
   )
+  (symbol (lib_id "PCM_Elektuur:C") (at 165.1 170.18 0) (unit 1)
+    (in_bom yes) (on_board yes) (dnp no) (fields_autoplaced)
+    (property "Reference" "C15" (at 168.91 168.91 0)
+      (effects (font (size 1.27 1.27)) (justify left))
+    )
+    (property "Value" "1uF" (at 168.91 171.45 0)
+      (effects (font (size 1.27 1.27)) (justify left))
+    )
+    (property "Footprint" "" (at 165.1 170.18 0)
+      (effects (font (size 1.27 1.27)) hide)
+    )
+    (property "Datasheet" "" (at 165.1 170.18 0)
+      (effects (font (size 1.27 1.27)) hide)
+    )
+    (property "Indicator" "+" (at 163.83 167.005 0)
+      (effects (font (size 1.27 1.27)) hide)
+    )
+    (property "Rating" "V" (at 164.465 173.355 0)
+      (effects (font (size 1.27 1.27)) (justify right) hide)
+    )
+    (pin "1")
+    (pin "2")
+    (instances
+      (project "filter"
+        (path "/69b3d959-9103-4d24-8a1d-6bf78309c8d1"
+          (reference "C15") (unit 1)
+        )
+      )
+    )
+  )
   (symbol (lib_id "PCM_Generic-50:C,IEC") (at 115.57 25.4 0) (mirror x) (unit 1)
     (in_bom yes) (on_board yes) (dnp no) (fields_autoplaced)
@@
         )
       )
+    )
+  )
+  (symbol (lib_id "PCM_Elektuur:R") (at 165.1 180.34 180) (unit 1)
+    (in_bom yes) (on_board yes) (dnp no) (fields_autoplaced)
+    (property "Reference" "R13" (at 168.275 179.07 0)
+      (effects (font (size 1.27 1.27)) (justify right))
+    )
+    (property "Value" "8 Om" (at 168.275 181.61 0)
+      (effects (font (size 1.27 1.27)) (justify right))
+    )
+    (property "Footprint" "" (at 165.1 180.34 0)
+      (effects (font (size 1.27 1.27)) hide)
+    )
+    (property "Datasheet" "" (at 165.1 180.34 0)
+      (effects (font (size 1.27 1.27)) hide)
+    )
+    (property "Indicator" "+" (at 168.275 183.515 0)
+      (effects (font (size 1.27 1.27)) hide)
+    )
+    (property "Rating" "W" (at 162.56 177.165 0)
+      (effects (font (size 1.27 1.27)) (justify left) hide)
+    )
+    (pin "1")
+    (pin "2")
+    (instances
+      (project "filter"
+        (path "/69b3d959-9103-4d24-8a1d-6bf78309c8d1"
+          (reference "R13") (unit 1)
+        )
+      )

Commit message: Upgrade
Parts:
- removed L1: L 1,ferrite-bead,IEC, symbol PCM_Generic:L,ferrite-bead,IEC
- removed L2: L 1, ferrite-bead,IEC, symbol PCM_Generic:L,ferrite-bead,IEC
- removed L3, L4: L 2, ferrite-bead,IEC, symbol PCM_Generic:L,ferrite-bead,IEC
- added C18: 1uF, symbol PCM_Elektuur:C
- added R18: 8 Om, symbol PCM_Elektuur:R
- added R24: 2.4, symbol PCM_Generic:R,IEC
- added R25: 10 Om, symbol PCM_Generic:R,IEC
- added R26: 1.5, symbol PCM_Generic:R,IEC
Connections:
- net PE: now also C18.1 (+), R18.1 (+), R24.2 (-), R25.2 (-), R26.2 (-)
- net at R23.2 (-): now also R11.2 (-), R12.2 (-), R15.2 (-), R17.2 (-), R19.2 (-), R22.2 (-), R4.2 (-), R5.2 (-), R6.2 (-), R7.2 (-), R24.1 (+), R25.1 (+), R26.1 (+)
- new net: C18.2 (-), R18.2 (-)
Other:
- note added: "??????????????????????"
- note added: "Home"
- note added: "an attempt to align the frequencies that led to the understanding that I was under the control of a Scientologist pirate"
- moved on the sheet: C11, C14, R11
