File: filter.kicad_sch (KiCad schematic)
At the start: 93 parts, among them U1 ${SIM.PARAMS}

Commit message: Upgrade
Parts:
- removed R7: 8 Om, symbol PCM_Generic:R,IEC
- added R28: 12 Om, symbol PCM_Generic:R,IEC
- R11: value 90 Om -> 47 Om
- R12: value 8 Om -> ~3 Om
Connections:
- net at C23.2 (-), C24.1 (+): now also R28.1 (+)
- net at R11.2 (-), R12.2 (-), R15.2 (-)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: now also R28.2 (-)
Other:
- note added: "3"
- note added: "Grounding devices"
- note added: "Same filters at 1.5-2 Km distance, without 30uF ELF filer"
- note removed: "Same filters at 1.5-2 Km distance"
Changed lines of the file:
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@@
 		)
 	)
-	(text_box "R1,R2,R8,R9,R12,R11,R16,R14,R27,R29,R25,R24 = 33KOm\nR3,R10,R13,R26,R21,R20 = 15KOm\nR4,R7,R15,R23,R30,R31,R33,R34,R35,R36 = 2-10MOm all dumping resistors must have same nominal ( 10MOm as example ) and model !!!!!\nR5,R6,R18,R15,R17,R22,R28,R32 = 7-10Om   R4,R19 = 50Om 2GHz about 450 W\nC1,C6,C9,C17,C16,C18 = 220nF\nC2,C3,C7,C8,C11,C10,C12,C13,C20,C19,C21,C22 = 100nF\nC15,C14 = 10-100 nF - optional, I use MC1230 | C4,C5 = 100 nF   C23,C24 = 35 mkF\nC25,C26, C27,C28 = 22 pF C9, C10 = 10 nF\n\ntry to keep maximum possible distance between filters ~ 30cm\n\nMC 1230 optional"
+	(text_box "R1,R2,R8,R9,R12,R11,R16,R14,R27,R29,R25,R24 = 33KOm\nR3,R10,R13,R26,R21,R20 = 15KOm\nR7,R15,R23,R30,R31,R33,R34,R35,R36 = 2-10MOm all dumping resistors must have same nominal ( 10MOm as example ) and model !!!!!\nR5,R6,R18,R15,R17,R22,R28,R32 = 7-10Om   R4,R19 = 50Om 2GHz about 450 W\nC1,C6,C9,C17,C16,C18 = 220nF\nC2,C3,C7,C8,C11,C10,C12,C13,C20,C19,C21,C22 = 100nF\nC15,C14 = 10-100 nF - optional, I use MC1230 | C4,C5 = 100 nF   C23,C24 = 35-30 mkF\nC25,C26, C27,C28 = 22 pF C9, C10 = 10 nF\n\ntry to keep maximum possible distance between filters ~ 30cm\n\nMC 1230 optional"
 		(exclude_from_sim no)
 		(at 13.97 152.4 0)
@@
 		)
 	)
+	(text "3 \n"
+		(exclude_from_sim no)
+		(at 135.89 136.398 0)
+		(effects
+			(font
+				(size 1.27 1.27)
+			)
+		)
+	)
 	(text "29.02.2024\n"
 		(exclude_from_sim no)
@@
 		)
 	)
-	(text "Grounding device"
+	(text "Grounding devices"
 		(exclude_from_sim no)
 		(at 137.16 137.16 0)
@@
 		)
 	)
-	(text "Same filters at 1.5-2 Km distance\n"
+	(text "Same filters at 1.5-2 Km distance, \nwithout 30uF ELF filer\n\n\n"
 		(exclude_from_sim no)
 		(at 241.3 95.25 0)
@@
 			)
 		)
-		(property "Value" "90 Om"
+		(property "Value" "47 Om"
 			(at 196.85 133.35 90)
 			(effects
@@
 			)
 		)
-		(property "Value" "8 Om"
+		(property "Value" "~3 Om"
 			(at 176.53 74.9299 0)
 			(effects
@@
 	)
 	(symbol
+		(lib_id "PCM_Generic:R,IEC")
+		(at 72.39 69.85 0)
+		(unit 1)
+		(exclude_from_sim no)
+		(in_bom yes)
+		(on_board yes)
+		(dnp no)
+		(fields_autoplaced yes)
+		(property "Reference" "R28"
+			(at 74.93 67.3099 0)
+			(effects
+				(font
+					(size 2.54 2.54)
+				)
+				(justify left)
+			)
+		)
+		(property "Value" "12 Om"
+			(at 74.93 72.3899 0)
+			(effects
+				(font
+					(size 2.54 2.54)
+				)
+				(justify left)
+			)
+		)
+		(property "Footprint" ""
+			(at 72.39 69.85 0)
+			(effects
+				(font
+					(size 2.54 2.54)
+				)
+				(hide yes)
+			)
+		)
+		(property "Datasheet" ""
+			(at 72.39 69.85 0)
+			(effects
+				(font
+					(size 2.54 2.54)
+				)
+				(hide yes)
+			)
+		)
+		(property "Description" ""
+			(at 72.39 69.85 0)
+			(effects
+				(font
+					(size 1.27 1.27)
+				)
+				(hide yes)
+			)
+		)
+		(property "Indicator" ""
+			(at 69.85 67.31 0)
+			(effects
+				(font
+					(size 1.27 1.27)
+				)
+				(hide yes)
+			)
+		)
+		(pin "1"
+		)
+		(pin "2"
+		)
+		(instances
+			(project "filter"
+				(path "/69b3d959-9103-4d24-8a1d-6bf78309c8d1"
+					(reference "R28")
+					(unit 1)
+				)
+			)
+		)
+	)
+	(symbol
 		(lib_id "PCM_Generic:C,IEC")
 		(at 205.74 142.24 0)
@@
 					(unit 1)
 				)
-			)
-		)
-	)
-	(symbol
-		(lib_id "PCM_Generic:R,IEC")
-		(at 72.39 69.85 0)
-		(unit 1)
-		(exclude_from_sim no)
-		(in_bom yes)
-		(on_board yes)
-		(dnp no)
-		(fields_autoplaced yes)
-		(property "Reference" "R7"
-			(at 74.93 67.3099 0)
-			(effects
-				(font
-					(size 2.54 2.54)
-				)
-				(justify left)
-			)
-		)
-		(property "Value" "8 Om"
-			(at 74.93 72.3899 0)
-			(effects
-				(font
-					(size 2.54 2.54)
-				)
-				(justify left)
-				(hide yes)
-			)
-		)
-		(property "Footprint" ""
-			(at 72.39 69.85 0)
-			(effects
-				(font
-					(size 2.54 2.54)
-				)
-				(hide yes)
-			)
-		)
-		(property "Datasheet" ""
-			(at 72.39 69.85 0)
-			(effects
-				(font
-					(size 2.54 2.54)
-				)
-				(hide yes)
-			)
-		)
-		(property "Description" ""
-			(at 72.39 69.85 0)
-			(effects
-				(font
-					(size 1.27 1.27)
-				)
-				(hide yes)
-			)
-		)
-		(property "Indicator" ""
-			(at 69.85 67.31 0)
-			(effects
-				(font
-					(size 1.27 1.27)
-				)
-				(hide yes)
-			)
-		)
-		(pin "1"
-		)
-		(pin "2"
-		)
-		(instances
-			(project "filter"
-				(path "/69b3d959-9103-4d24-8a1d-6bf78309c8d1"
-					(reference "R7")
-					(unit 1)
-				)

Commit message: Upgrade
Parts:
- added C19, C32: C,220nF, symbol PCM_Generic:C,IEC
- added C20, C33, C34: C,100nF, symbol PCM_Generic-50:C,IEC
- added C29: C, 100nF, symbol PCM_Generic-50:C,IEC
- added C30, C31: C,1 mkF, symbol PCM_Generic:C,IEC
- added E1: SparkGap, symbol Device:SparkGap
- added R30: R,33kOm, symbol PCM_Generic:R,IEC
- added R31: R,15kOm, symbol PCM_Generic:R,IEC
- added R7: R, 33kOm, symbol PCM_Generic:R,IEC
- C23, C24: value C,IEC -> C, 60 mkF
- R12: value ~3 Om -> 2 Om
- R17: value 10 Om -> R,15kOm; Indicator (none) -> +
- R22: value 8 Om -> 2 Om
- R23: value 8 Om -> 0.5 Om
- R24: value 2.4 -> 10 Om
- R25: value 10 Om -> 2 Om
- R26: value 1.5 -> R,33kOm; Indicator (none) -> +
- R28: value 12 Om -> 3 Om
- R6: value 10 Om -> R,33kOm; Indicator (none) -> +
Connections:
- net PE: now also E1.2; no longer R24.2 (-), R25.2 (-), R26.2 (-)
- net at C23.2 (-), C24.1 (+), R28.1 (+): now also R28.2 (-), R5.2 (-)
- net at C16.2 (-), C17.2 (-), R20.1 (+)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: no longer R6.1 (+)
- net at C1.2 (-), C6.2 (-), R10.1 (+)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: no longer R17.1 (+)
- net at R11.2 (-), R12.2 (-), R15.2 (-)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: now also R24.2 (-), R25.2 (-); no longer R17.2 (-), R24.1 (+), R25.1 (+), R26.1 (+), R28.2 (-), R5.2 (-), R6.2 (-)
- new net: C19.2 (-), C32.2 (-), R17.1 (+), R24.1 (+), R31.1 (+)
- new net: C33.1 (+), C34.2 (-), R31.2 (-)
- new net: C20.2 (-), C30.1 (+), R6.2 (-)
- new net: C30.2 (-), C31.1 (+), R25.1 (+)
- new net: C31.2 (-), C33.2 (-), R26.2 (-)
- new net: C29.1 (+), R7.1 (+)
- new net: C20.1 (+), C29.2 (-), R17.2 (-)
- new net: C19.1 (+), R6.1 (+), R7.2 (-)
- new net: C34.1 (+), R30.1 (+)
- new net: C32.1 (+), R26.1 (+), R30.2 (-)
Other:
- note added: "2"
- note added: "5m distance"
- note added: "Optional, experimental"
- note added: "Same filters at 1.5-2 Km distance, without 60uF ELF filer"
- note removed: "3"
- note removed: "??????????????????????"
- note removed: "Same filters at 1.5-2 Km distance, without 30uF ELF filer"
- note removed: "an attempt to align the frequencies that led to the understanding that I was under the control of a Scientologist pirate"
- moved on the sheet: C1, C12, C13, C16, C17, C2, C21, C22, C23, C24, C3, C4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

Commit message: Upgrade
Parts:
- added E2: SparkGap, symbol Device:SparkGap
- C23, C24: value C, 60 mkF -> C, 80 mkF
- C30, C31: value C,1 mkF -> C,0.8mkF
- R13, R18: value 8 Om -> 2 Om
- R28: value 3 Om -> 2 Om
Connections:
- net PE: now also E2.2
- net at C23.2 (-), C24.1 (+), R28.1 (+): no longer R28.2 (-), R5.2 (-)
- new net: R28.2 (-), R5.2 (-)
Changed lines of the file:
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@@
 	)
 	(junction
+		(at 68.58 97.79)
+		(diameter 0)
+		(color 0 0 0 0)
+	)
+	(junction
 		(at 217.17 16.51)
 		(diameter 0)
@@
 	)
 	(junction
-		(at 58.42 60.96)
-		(diameter 0)
-		(color 0 0 0 0)
-	)
-	(junction
 		(at 165.1 128.27)
 		(diameter 0)
@@
 	(wire
 		(pts
+			(xy 68.58 97.79) (xy 68.58 107.95)
+		)
+		(stroke
+			(width 0)
+			(type default)
+		)
+	)
+	(wire
+		(pts
 			(xy 139.7 16.51) (xy 170.18 16.51)
 		)
@@
 	(wire
 		(pts
+			(xy 52.07 107.95) (xy 52.07 113.03)
+		)
+		(stroke
+			(width 0)
+			(type default)
+		)
+	)
+	(wire
+		(pts
 			(xy 87.63 54.61) (xy 97.79 54.61)
 		)
@@
 	(wire
 		(pts
+			(xy 62.23 107.95) (xy 68.58 107.95)
+		)
+		(stroke
+			(width 0)
+			(type default)
+		)
+	)
+	(wire
+		(pts
 			(xy 139.7 38.1) (xy 139.7 44.45)
 		)
@@
 	(wire
 		(pts
-			(xy 62.23 97.79) (xy 78.74 97.79)
+			(xy 62.23 97.79) (xy 68.58 97.79)
 		)
 		(stroke
@@
 	(wire
 		(pts
+			(xy 68.58 97.79) (xy 78.74 97.79)
+		)
+		(stroke
+			(width 0)
+			(type default)
+		)
+	)
+	(wire
+		(pts
 			(xy 398.78 106.68) (xy 412.75 106.68)
 		)
@@
 	(wire
 		(pts
-			(xy 58.42 44.45) (xy 58.42 60.96)
-		)
-		(stroke
-			(width 0)
-			(type default)
-		)
-	)
-	(wire
-		(pts
 			(xy 125.73 128.27) (xy 69.85 128.27)
 		)
@@
 	(wire
 		(pts
-			(xy 58.42 60.96) (xy 58.42 77.47)
+			(xy 58.42 44.45) (xy 58.42 77.47)
 		)
 		(stroke
@@
 		)
 	)
-	(text_box "R1,R2,R8,R9,R12,R11,R16,R14,R27,R29,R25,R24 = 33KOm\nR3,R10,R13,R26,R21,R20 = 15KOm\nR7,R15,R23,R30,R31,R33,R34,R35,R36 = 2-10MOm all dumping resistors must have same nominal ( 10MOm as example ) and model !!!!!\nR5,R6,R18,R15,R17,R22,R28,R32 = 7-10Om   R4,R19 = 50Om 2GHz about 450 W\nC1,C6,C9,C17,C16,C18 = 220nF\nC2,C3,C7,C8,C11,C10,C12,C13,C20,C19,C21,C22 = 100nF\nC4,C5 = 100 nF   C23,C24 = 60 mkF\nC25,C26, C27,C28 = 22 pF C9, C10 = 10 nF\n\ntry to keep maximum possible distance between filters ~ 30cm\n\nMC 1230 optional"
+	(text_box "R1,R2,R8,R9,R12,R11,R16,R14,R27,R29,R25,R24 = 33KOm\nR3,R10,R13,R26,R21,R20 = 15KOm\nR7,R15,R23,R30,R31,R33,R34,R35,R36 = 2-10MOm all dumping resistors must have same nominal ( 10MOm as example ) and model !!!!!\nR5,R6,R18,R15,R17,R22,R28,R32 = 7-10Om   R4,R19 = 50Om 2GHz about 450 W\nC1,C6,C9,C17,C16,C18 = 220nF\nC2,C3,C7,C8,C11,C10,C12,C13,C20,C19,C21,C22 = 100nF\nC4,C5 = 82 nF   C23,C24 = 60 mkF\nC25,C26, C27,C28 = 22 pF C9, C10 = 10 nF\n\ntry to keep maximum possible distance between filters ~ 30cm\n\nMC 1230 optional"
 		(exclude_from_sim no)
 		(at 13.97 152.4 0)
@@
 			)
 		)
-		(property "Value" "C, 60 mkF"
+		(property "Value" "C, 80 mkF"
 			(at 51.562 64.77 90)
 			(effects
@@
 			)
 		)
-		(property "Value" "C,1 mkF"
+		(property "Value" "C,0.8mkF"
 			(at 221.742 62.992 90)
 			(effects
@@
 			)
 		)
-		(property "Value" "C,1 mkF"
+		(property "Value" "C,0.8mkF"
 			(at 245.872 69.088 0)
 			(effects
@@
 			)
 		)
-		(property "Value" "3 Om"
+		(property "Value" "2 Om"
 			(at 71.12 72.3899 0)
 			(effects
@@
 	)
 	(symbol
+		(lib_id "Device:SparkGap")
+		(at 57.15 107.95 0)
+		(unit 1)
+		(exclude_from_sim no)
+		(in_bom yes)
+		(on_board yes)
+		(dnp no)
+		(fields_autoplaced yes)
+		(property "Reference" "E2"
+			(at 57.15 102.87 0)
+			(effects
+				(font
+					(size 1.27 1.27)
+				)
+			)
+		)
+		(property "Value" "SparkGap"
+			(at 57.15 105.41 0)
+			(effects
+				(font
+					(size 1.27 1.27)
+				)
+			)
+		)
+		(property "Footprint" ""
+			(at 57.15 109.728 0)
+			(effects
+				(font
+					(size 1.27 1.27)
+				)
+				(hide yes)
+			)
+		)
+		(property "Datasheet" "~"
+			(at 57.15 107.95 90)
+			(effects
+				(font
+					(size 1.27 1.27)
+				)
+				(hide yes)
+			)
+		)
+		(property "Description" "Spark gap"
+			(at 57.15 107.95 0)
+			(effects
+				(font
+					(size 1.27 1.27)
+				)
+				(hide yes)
+			)
+		)
+		(pin "2"
+		)
+		(pin "1"
+		)
+		(instances
+			(project "filter"
+				(path "/69b3d959-9103-4d24-8a1d-6bf78309c8d1"
+					(reference "E2")
+					(unit 1)
+				)
+			)
+		)
+	)
+	(symbol
 		(lib_id "PCM_Generic:C,IEC")
 		(at 205.74 142.24 0)
@@
 			)
 		)
-		(property "Value" "C, 60 mkF"
+		(property "Value" "C, 80 mkF"
 			(at 71.12 66.294 0)
 			(effects
@@
 		(fields_autoplaced yes)
 		(property "Reference" "R13"
-			(at 168.275 179.07 0)
+			(at 167.64 179.0699 0)
 			(effects
 				(font
@@
 			)
 		)
-		(property "Value" "8 Om"
-			(at 168.275 181.61 0)
+		(property "Value" "2 Om"
+			(at 167.64 181.6099 0)
 			(effects
 				(font
@@
 		(fields_autoplaced yes)
 		(property "Reference" "R18"
-			(at 260.985 147.32 0)
+			(at 260.35 147.3199 0)
 			(effects
 				(font
@@
 			)
 		)
-		(property "Value" "8 Om"
-			(at 260.985 149.86 0)
+		(property "Value" "2 Om"
+			(at 260.35 149.8599 0)
 			(effects
 				(font

Commit message: Upgrade
Parts:
- added C35, C36: C,220pF, symbol PCM_Generic:C,IEC
- added R32: 2Om, symbol PCM_Generic:R,IEC
Connections:
- net at R11.2 (-), R12.2 (-), R15.2 (-)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: now also R32.2 (-)
- new net: C35.2 (-), C36.1 (+), R32.1 (+)

Commit message: Upgarde
Parts:
- removed C15, C18: 1uF, symbol PCM_Elektuur:C
- removed R13, R18: 2 Om, symbol PCM_Elektuur:R
- removed R15, R24: 10 Om, symbol PCM_Generic:R,IEC
- removed R23: 0.5 Om, symbol PCM_Generic:R,IEC
- added C15: C, 200 pf, symbol PCM_Generic:C,IEC
- added C18: C,200 pF, symbol PCM_Generic:C,IEC
- added C37, C38: C, symbol Device:C
- added L1: L 10-15 coil turn, symbol Device:L_Ferrite_Coupled_Small
- C11, C14: value C,22pF -> C,200pF
- C23, C24: value C, 80 mkF -> C, 880 mkF
- R11: value 47 Om -> 1 Om
- R5: value 10 Om -> 1 Om
Connections:
- net at R11.2 (-), R12.2 (-), R19.2 (-)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: now also R5.2 (-)
- net at C16.2 (-), C17.2 (-), R20.1 (+)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: no longer R5.1 (+)
- net at R28.2 (-): no longer R5.2 (-)
- new net: C15.2 (-), C18.1 (+), R5.1 (+)
- new net in: C37.1, C38.2, L1.1, L1.3
- new net out: C37.2, C38.1, L1.2, L1.4
Other:
- note added: "01.06.2024"
- note added: "Installed on the power supply line of the devices where the power cable is connected. Just install multiple filters: 1 filter with C1,C2 - 10mkF, 1 filter with C1,C2 - 30mkF, 1 filter with C1,C2 - 680nF, 1 filter with C1,C2 - 8,2nF, 1 filter with C1,C2 - 100nF, 1 filter with C1,C2 - 220nF, 1 filter with C1,C2 - 80nF"
- note added: "Optional, experimental, WIP"
- note added: "Same filters at 2 Km distance, separated by LPT-s without 880uF ELF filer"
- note removed: "29.02.2024"
- note removed: "MC 1230"
- note removed: "Optional, experimental"
- note removed: "Same filters at 1.5-2 Km distance, without 60uF ELF filer"
- note removed: "They say this is idea from life of Tupak -_^^_-"

Commit message: Upgarade
Parts:
- added C39, C40: C, symbol Device:C
- added L2: L 10-15 coil turn, symbol Device:L_Ferrite_Coupled_Small
Connections:
- net in: now also C39.1; no longer C38.2, L1.1
- net out: now also C38.2, C40.1, L2.3; no longer C38.1
- new net: C39.2, L2.4
- new net: C40.2, L2.2
- new net in Line: C38.1, L1.1, L2.1
Other:
- note added: "Installed on the power supply line of the devices where the power cable is connected. Just install multiple filters: 1 filter with C1,C2 - 10mkF, 1 filter with C1,C2 - 30mkF, 1 filter with C1,C2 - 680nF, 1 filter with C1,C2 - 8,2nF, 1 filter with C1,C2 - 100nF, 1 filter with C1,C2 - 220nF, 1 filter with C1,C2 - 80nF, 4 filters with C1,C2 - 1nF"
- note removed: "Installed on the power supply line of the devices where the power cable is connected. Just install multiple filters: 1 filter with C1,C2 - 10mkF, 1 filter with C1,C2 - 30mkF, 1 filter with C1,C2 - 680nF, 1 filter with C1,C2 - 8,2nF, 1 filter with C1,C2 - 100nF, 1 filter with C1,C2 - 220nF, 1 filter with C1,C2 - 80nF"
- moved on the sheet: C37, C38

Commit message: Upgrade
Parts:
- removed C37, C38, C39, C40: C, symbol Device:C
- removed L1, L2: L 10-15 coil turn, symbol Device:L_Ferrite_Coupled_Small
- added C37, C38: 1mkF, symbol Device:C_Small
- added C39, C40, C46, C47: 220nF, symbol Device:C_Small
- added C41: From 1mkF to 10 nF, symbol Device:C_Small
- added C42, C43: C_Small, symbol Device:C_Small
- added C44, C45: 10mkF, symbol Device:C_Small
- added C48, C49: 100nF, symbol Device:C_Small
- added C50, C51: 10nF, symbol Device:C_Small
- added L1, L2, L3, L4, L5, L7, L8, L9: L_ferrite, symbol Device:L_Coupled
- added L10, L11: ~, symbol Device:L_Ferrite_Small
- added L6: Ferrite, symbol Device:L
- added R13, R15, R18, R23: 2Om, symbol Device:R_Small
Connections:
- net out: now also C44.2, C45.2, L2.1, L2.3
- new net: C39.1, L4.2, L5.1
- new net: C39.2, L4.4, L5.3
- new net: C41.1, L10.2, L6.1
- new net: C41.2, L1.4, L11.1
- new net: C38.1, C46.2, L3.2, L4.1
- new net: C38.2, C47.2, L3.4, L4.3
- new net: C37.1, L2.2, L3.1
- new net: C37.2, L2.4, L3.3
- new net: C50.1, C51.1, R13.2
- new net: C51.2, L11.2, L8.3
- new net: C48.1, C49.1, R15.2
- new net: C40.2, C48.2, L5.4, L9.2
- new net: C46.1, C47.1, R18.2
- new net: C40.1, C49.2, L5.2, L9.4
- new net: C43.1, L7.2, L9.1
- new net: C43.2, L7.4, L9.3
- new net: C42.1, L7.1, L8.2
- new net: C42.2, L7.3, L8.4
- new net: R13.1, R15.1, R18.1, R23.1
- new net: C44.1, C45.1, R23.2
- new net: C50.2, L10.1, L8.1
- new net: L1.2, L6.2
Other:
- note added: "Dc light, routhers, osciloscopes"
- note added: "Filter with phase shift"
- note removed: "Installed on the power supply line of the devices where the power cable is connected. Just install multiple filters: 1 filter with C1,C2 - 10mkF, 1 filter with C1,C2 - 30mkF, 1 filter with C1,C2 - 680nF, 1 filter with C1,C2 - 8,2nF, 1 filter with C1,C2 - 100nF, 1 filter with C1,C2 - 220nF, 1 filter with C1,C2 - 80nF, 4 filters with C1,C2 - 1nF"

Commit message: Upgrade
Parts:
- R12: value 2 Om -> 10 Om
Other:
- moved on the sheet: R25
Changed lines of the file:
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@@
 	(wire
 		(pts
-			(xy 251.46 78.74) (xy 190.5 78.74)
+			(xy 250.19 77.47) (xy 209.55 77.47)
 		)
 		(stroke
@@
 	(wire
 		(pts
-			(xy 231.14 74.93) (xy 231.14 76.2)
+			(xy 231.14 72.39) (xy 231.14 73.66)
 		)
 		(stroke
@@
 	(wire
 		(pts
-			(xy 231.14 58.42) (xy 231.14 64.77)
+			(xy 231.14 58.42) (xy 231.14 62.23)
 		)
 		(stroke
@@
 	(wire
 		(pts
-			(xy 251.46 52.07) (xy 251.46 78.74)
+			(xy 250.19 52.07) (xy 250.19 77.47)
 		)
 		(stroke
@@
 	(wire
 		(pts
-			(xy 231.14 52.07) (xy 251.46 52.07)
+			(xy 231.14 52.07) (xy 250.19 52.07)
 		)
 		(stroke
@@
 	(wire
 		(pts
-			(xy 217.17 76.2) (xy 217.17 127)
+			(xy 217.17 73.66) (xy 217.17 127)
 		)
 		(stroke
@@
 	(wire
 		(pts
-			(xy 217.17 76.2) (xy 231.14 76.2)
+			(xy 217.17 73.66) (xy 231.14 73.66)
 		)
 		(stroke
@@
 	(wire
 		(pts
-			(xy 190.5 78.74) (xy 190.5 83.82)
+			(xy 209.55 77.47) (xy 209.55 83.82)
 		)
 		(stroke
@@
 		)
 	)
-	(text_box "R1,R2,R8,R9,R12,R11,R16,R14,R27,R29,R25,R24 = 33KOm\nR3,R10,R13,R26,R21,R20 = 15KOm\nR5,R6,R18,R15,R17,R22,R28,R32 = 7-10Om   R4,R19 = 50Om 2GHz about 450 W\nC1,C6,C9,C17,C16,C18 = 220nF\nC2,C3,C7,C8,C11,C10,C12,C13,C20,C19,C21,C22 = 100nF\nC4,C5 = 82 nF   C23,C24 = 880 mkF\nC25,C26, C27,C28 = 9 pF C9, C10 = 10 nF\n\ntry to keep maximum possible distance between filters ~ 30cm\n\nMC 1230 optional"
+	(text_box "R1,R2,R8,R9,R12,R11,R16,R14,R27,R29,R25,R24 = 33KOm\nR3,R10,R13,R26,R21,R20 = 15KOm\nR5,R6,R18,R15,R17,R22,R28,R32 = 7-10Om   R4,R19 = 50Om 2GHz about 450 W\nC1,C6,C9,C17,C16,C18 = 220nF\nC2,C3,C7,C8,C11,C10,C12,C13,C20,C19,C21,C22 = 100nF\nC4,C5 = 1.6 nF   C23,C24 = 880 mkF\nC25,C26, C27,C28 = 9 pF C9, C10 = 10 nF\n\ntry to keep maximum possible distance between filters ~ 30cm\n\nMC 1230 optional"
 		(exclude_from_sim no)
 		(at 13.97 152.4 0)
@@
 	(symbol
 		(lib_id "PCM_Generic:R,IEC")
-		(at 231.14 69.85 0)
+		(at 231.14 67.31 0)
 		(unit 1)
 		(exclude_from_sim no)
@@
 		(fields_autoplaced yes)
 		(property "Reference" "R25"
-			(at 233.68 67.3099 0)
+			(at 233.68 64.7699 0)
 			(effects
 				(font
@@
 		)
 		(property "Value" "2 Om"
-			(at 233.68 72.3899 0)
+			(at 233.68 69.8499 0)
 			(effects
 				(font
@@
 		)
 		(property "Footprint" ""
-			(at 231.14 69.85 0)
+			(at 231.14 67.31 0)
 			(effects
 				(font
@@
 		)
 		(property "Datasheet" ""
-			(at 231.14 69.85 0)
+			(at 231.14 67.31 0)
 			(effects
 				(font
@@
 		)
 		(property "Description" ""
-			(at 231.14 69.85 0)
+			(at 231.14 67.31 0)
 			(effects
 				(font
@@
 		)
 		(property "Indicator" ""
-			(at 228.6 67.31 0)
+			(at 228.6 64.77 0)
 			(effects
 				(font
@@
 			)
 		)
-		(property "Value" "2 Om"
+		(property "Value" "10 Om"
 			(at 144.78 72.3899 0)
 			(effects
